File: JANUSJFH/JANUSJFH.kicad_sch (KiCad schematic)
At the start: 30 parts, among them J1 USB_B_Micro, SW1 SW_SPDT, U1 STM32L476RGTx, U2 AMS1117-3.3, U3 BMP280, U4 IP4234CZ6

Commit message: Add files via upload
Parts:
- removed U4: IP4234CZ6, Package_TO_SOT_SMD:SC-74-6_1.55x2.9mm_P0.95mm, symbol Power_Protection:IP4234CZ6
Connections:
- net I2C1_SCL: now also R5.1, U1.59 (PB7); no longer R4.1, U1.58 (PB6)
- net I2C1_SDA: now also R4.1, U1.58 (PB6); no longer R5.1, U1.59 (PB7)
- net USB_OTG_FS_DM-: now also J1.2 (D-)
- net USB_OTG_FS_DP+: now also J1.3 (D+)
Other:
- moved on the sheet: R4, R5
